File: electronics/opto-isolator/Prueba.kicad_pcb (KiCad board)
At the start: 2 copper layers, 4 parts, among them P1 CONN_01X03

Commit message: Electronics update
Routing:
- net GND: track 38.9 -> 0.00 mm
- net VCC: track 41.6 -> 28.2 mm
- net /Signal: track 22.9 -> 28.4 mm
- added copper zone on B.Cu, net GND
Other:
- board outline added: 36 x 15.5 mm
- net class Default: clearance 0.2 -> 0.635; trace_width 0.25 -> 1.27
- rule trace_clearance: 0.2 -> 0.635
