File: electronics/ControlPCB/_saved_ControlPCB.sch (KiCad schematic (older format))
At the start: 70 parts, among them CON1 12VINPUT, P1 CONN_02X03, P2 CONN_02X03, P3 CONN_02X03, P4 CONN_02X03, P5 CONN_02X03, P6 CONN_02X03, P7 CONN_02X03, P8 CONN_02X03, U1 POLOLU_A4988, U2 POLOLU_A4988, U3 POLOLU_A4988, U4 POLOLU_A4988, U5 POLOLU_A4988, U6 POLOLU_A4988, U7 POLOLU_A4988, U8 POLOLU_A4988

Commit message: ControlPCB before square
Connections:
- net STEPM1: now also PDIG1.9 (P9); no longer PDIG1.3 (P3)
- net STEPM2: now also PDIG1.7 (P7); no longer PDIG1.4 (P4)
- net STEPM4: now also PDIG1.3 (P3); no longer PDIG1.6 (P6)
- net STEPM5: now also PDIG1.4 (P4); no longer PDIG1.7 (P7)
- net STEPM6: now also PDIG1.6 (P6); no longer PDIG1.8 (P8)
- net STEPM7: now also PDIG1.8 (P8); no longer PDIG1.9 (P9)
- net VCC: now also P1.2 (P2), P1.4 (P4), P1.6 (P6), P2.2 (P2), P2.4 (P4), P2.6 (P6), P3.2 (P2), P3.4 (P4), P3.6 (P6), P4.2 (P2), P4.4 (P4), P4.6 (P6), P5.2 (P2), P5.4 (P4), P5.6 (P6), P6.2 (P2), P6.4 (P4), P6.6 (P6), P7.2 (P2), P7.4 (P4), P7.6 (P6), P8.2 (P2), P8.4 (P4), P8.6 (P6); no longer P1.1 (P1), P1.3 (P3), P1.5 (P5), P2.1 (P1), P2.3 (P3), P2.5 (P5), P3.1 (P1), P3.3 (P3), P3.5 (P5), P4.1 (P1), P4.3 (P3), P4.5 (P5), P5.1 (P1), P5.3 (P3), P5.5 (P5), P6.1 (P1), P6.3 (P3), P6.5 (P5), P7.1 (P1), P7.3 (P3), P7.5 (P5), P8.1 (P1), P8.3 (P3), P8.5 (P5)
- net at R9.1, U1.10 (MS1): now also P1.5 (P5); no longer P1.2 (P2)
- net at U1.11 (MS2): now also P1.3 (P3); no longer P1.4 (P4)
- net at U1.12 (MS3): now also P1.1 (P1); no longer P1.6 (P6)
- net at R10.1, U2.10 (MS1): now also P2.5 (P5); no longer P2.2 (P2)
- net at U2.11 (MS2): now also P2.3 (P3); no longer P2.4 (P4)
- net at U2.12 (MS3): now also P2.1 (P1); no longer P2.6 (P6)
- net at R11.1, U3.10 (MS1): now also P3.5 (P5); no longer P3.2 (P2)
- net at U3.11 (MS2): now also P3.3 (P3); no longer P3.4 (P4)
- net at U3.12 (MS3): now also P3.1 (P1); no longer P3.6 (P6)
- net at R12.1, U4.10 (MS1): now also P4.5 (P5); no longer P4.2 (P2)
- net at U4.11 (MS2): now also P4.3 (P3); no longer P4.4 (P4)
- net at U4.12 (MS3): now also P4.1 (P1); no longer P4.6 (P6)
- net at R13.1, U5.10 (MS1): now also P5.5 (P5); no longer P5.2 (P2)
- net at U5.11 (MS2): now also P5.3 (P3); no longer P5.4 (P4)
- net at U5.12 (MS3): now also P5.1 (P1); no longer P5.6 (P6)
- net at R14.1, U6.10 (MS1): now also P6.5 (P5); no longer P6.2 (P2)
- net at U6.11 (MS2): now also P6.3 (P3); no longer P6.4 (P4)
- net at U6.12 (MS3): now also P6.1 (P1); no longer P6.6 (P6)
- net at R15.1, U7.10 (MS1): now also P7.5 (P5); no longer P7.2 (P2)
- net at U7.11 (MS2): now also P7.3 (P3); no longer P7.4 (P4)
- net at U7.12 (MS3): now also P7.1 (P1); no longer P7.6 (P6)
- net at R16.1, U8.10 (MS1): now also P8.5 (P5); no longer P8.2 (P2)
- net at U8.11 (MS2): now also P8.3 (P3); no longer P8.4 (P4)
- net at U8.12 (MS3): now also P8.1 (P1); no longer P8.6 (P6)
Changed lines of the file:
@@
 $EndComp
 Text GLabel 9750 2450 0    60   Output ~ 0
-STEPM1
+STEPM4
 Text GLabel 9750 2850 0    60   Output ~ 0
 DIRM1
@@
 DIRM3
 Text GLabel 9750 2650 0    60   Output ~ 0
-STEPM5
+STEPM2
 Text GLabel 9750 3050 0    60   Output ~ 0
 DIRM5
 Text GLabel 9750 2750 0    60   Output ~ 0
-STEPM7
+STEPM1
 Text GLabel 9750 3150 0    60   Output ~ 0
 DIRM7
 Text GLabel 10450 2450 2    60   Output ~ 0
-STEPM2
+STEPM5
 Text GLabel 10450 2850 2    60   Output ~ 0
 DIRM2
 Text GLabel 10450 2550 2    60   Output ~ 0
-STEPM4
+STEPM6
 Text GLabel 10450 2950 2    60   Output ~ 0
 DIRM4
 Text GLabel 10450 2650 2    60   Output ~ 0
-STEPM6
+STEPM7
 Text GLabel 10450 3050 2    60   Output ~ 0
 DIRM6
@@
 F 3 "" H 4700 3950 50  0000 C CNN
 	1    4700 5150
-	1    0    0    -1
+	-1   0    0    1
 $EndComp
 $Comp
@@
 F 3 "" H 4700 2650 50  0000 C CNN
 	1    4700 3850
-	1    0    0    -1
+	-1   0    0    1
 $EndComp
 $Comp
@@
 F 3 "" H 4700 1400 50  0000 C CNN
 	1    4700 2600
-	1    0    0    -1
+	-1   0    0    1
 $EndComp
 $Comp
@@
 F 3 "" H 1150 1400 50  0000 C CNN
 	1    1150 2600
-	1    0    0    -1
+	-1   0    0    1
 $EndComp
 $Comp
@@
 F 3 "" H 1150 2650 50  0000 C CNN
 	1    1150 3850
-	1    0    0    -1
+	-1   0    0    1
 $EndComp
 $Comp
@@
 F 3 "" H 1150 3950 50  0000 C CNN
 	1    1150 5150
-	1    0    0    -1
+	-1   0    0    1
 $EndComp
 $Comp
@@
 F 3 "" H 1150 100 50  0000 C CNN
 	1    1150 1300
-	1    0    0    -1
+	-1   0    0    1
 $EndComp
 $Comp
@@
 F 3 "" H 4700 100 50  0000 C CNN
 	1    4700 1300
-	1    0    0    -1
-$EndComp
-$Comp
+	-1   0    0    1
+$EndComp
+$Comp
