File: electronics/ControlPCB/ControlPCB.sch (KiCad schematic (older format))
At the start: 70 parts, among them P1 CONN_02X03, P2 CONN_02X03, P3 CONN_02X03, P4 CONN_02X03, P5 CONN_02X03, P6 CONN_02X03, P7 CONN_02X03, P8 CONN_02X03, U1 POLOLU_A4988, U2 POLOLU_A4988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

Commit message: Electronics schematics
Parts:
- R1, R2, R3, R4, R5, R6, R7, R8: value R -> 10k
- R10, R11, R12, R13, R14, R15, R16, R9: value R -> 100k
